File: Hardware/Tamagotchi-thing/Tamagotchi-thing.kicad_sch (KiCad schematic)
At the start: 18 parts, among them J2 Conn_01x04, J3 Conn_01x04, J4 USB_C_Receptacle_USB2.0, Q1 DMG3415U, SW5 SW_SPDT_321, U101 TPS63802DLAR, U2 USBLC6-2P6

Commit message: schematic work
Parts:
- removed BT1: Battery, Bongo-Cat-Fidget-Toy:BAT-TH_CR2032-BS-6-1, symbol Device:Battery
- removed C1: 10u, Capacitor_SMD:C_0603_1608Metric, symbol Device:C_Small
- removed C2: 22u, Capacitor_SMD:C_0603_1608Metric, symbol Device:C_Small
- removed D1, D3: D_Schottky, Diode_SMD:D_SOD-123F, symbol Device:D_Schottky
- removed J2, J3: Conn_01x04, Connector_PinHeader_2.54mm:PinHeader_1x04_P2.54mm_Horizontal, symbol Connector_Generic:Conn_01x04
- removed L102: 0.47uH, Inductor_SMD_Wurth:L_Wurth_WE-LQSH-2010, symbol Device:L
- removed Q1: DMG3415U, Package_TO_SOT_SMD:SOT-23, symbol Device:Q_PMOS_GSD
- removed R4: 91k, Resistor_SMD:R_0603_1608Metric, symbol Device:R_Small_US
- removed R5: 10k, Resistor_SMD:R_0603_1608Metric, symbol Device:R
- removed R6: 511k, Resistor_SMD:R_0603_1608Metric, symbol Device:R_Small_US
- removed SW5: SW_SPDT_321, Bongo-Cat-Fidget-Toy:SW-SMD_SK-3245S-L1-A-1, symbol Switch:SW_SPDT_321
- removed U101: TPS63802DLAR, Bongo-Cat-Fidget-Toy:VREG_TPS63802DLAR, symbol Bongo-Cat-Fidget-Toy:TPS63802DLAR
Other:
- sheet mcu renamed MCU
- added sheet Power (sch/power.kicad_sch)

Commit message: Schematic work
Parts:
- removed J4: USB_C_Receptacle_USB2.0, Connector_USB:USB_C_Receptacle_HCTL_HC-TYPE-C-16P-01A, symbol Connector:USB_C_Receptacle_USB2.0
- removed R1, R7: 5.1k, Resistor_SMD:R_0603_1608Metric, symbol Device:R
- removed U2: USBLC6-2P6, Package_TO_SOT_SMD:SOT-666, symbol Power_Protection:USBLC6-2P6
Other:
- sheet MCU ports: added LCD2_A0, LCD2_BL_EN, LCD2_CS, LCD2_RES, LCD2{I2C}, LCD_BL_EN, LCD{LCD}, OLED_RST, OLED{I2C}; removed none
- sheet OLED ports: added LCD2_A0, LCD2_BL_EN, LCD2_CS, LCD2_RES, LCD2{I2C}, LCD_BL_EN, LCD{LCD}, OLED_RST, OLED{I2C}; removed none

Commit message: Schematic and layout work
Other:
- company: (none) -> Afonso Muralha
- title: (none) -> Tamagotchi Thing
Changed lines of the file:
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@@
 	(generator_version "9.0")
 	(paper "A4")
+	(title_block
+		(title "Tamagotchi Thing")
+		(date "2025-07-15")
+		(rev "V0.1")
+		(company "Afonso Muralha")
+	)
 	(bus
 		(pts
-			(xy 125.73 106.68) (xy 134.62 106.68)
+			(xy 138.43 105.41) (xy 147.32 105.41)
 		)
 		(stroke
@@
 	(bus
 		(pts
-			(xy 125.73 100.33) (xy 134.62 100.33)
-		)
-		(stroke
-			(width 0)
-			(type default)
-		)
-	)
-	(wire
-		(pts
-			(xy 125.73 115.57) (xy 134.62 115.57)
-		)
-		(stroke
-			(width 0)
-			(type default)
-		)
-	)
-	(wire
-		(pts
-			(xy 125.73 118.11) (xy 134.62 118.11)
-		)
-		(stroke
-			(width 0)
-			(type default)
-		)
-	)
-	(wire
-		(pts
-			(xy 125.73 102.87) (xy 134.62 102.87)
-		)
-		(stroke
-			(width 0)
-			(type default)
-		)
-	)
-	(wire
-		(pts
-			(xy 125.73 120.65) (xy 134.62 120.65)
-		)
-		(stroke
-			(width 0)
-			(type default)
-		)
-	)
-	(wire
-		(pts
-			(xy 125.73 123.19) (xy 134.62 123.19)
-		)
-		(stroke
-			(width 0)
-			(type default)
-		)
-	)
-	(wire
-		(pts
-			(xy 125.73 109.22) (xy 134.62 109.22)
+			(xy 138.43 99.06) (xy 147.32 99.06)
+		)
+		(stroke
+			(width 0)
+			(type default)
+		)
+	)
+	(wire
+		(pts
+			(xy 138.43 114.3) (xy 147.32 114.3)
+		)
+		(stroke
+			(width 0)
+			(type default)
+		)
+	)
+	(wire
+		(pts
+			(xy 138.43 116.84) (xy 147.32 116.84)
+		)
+		(stroke
+			(width 0)
+			(type default)
+		)
+	)
+	(wire
+		(pts
+			(xy 138.43 101.6) (xy 147.32 101.6)
+		)
+		(stroke
+			(width 0)
+			(type default)
+		)
+	)
+	(wire
+		(pts
+			(xy 138.43 119.38) (xy 147.32 119.38)
+		)
+		(stroke
+			(width 0)
+			(type default)
+		)
+	)
+	(wire
+		(pts
+			(xy 138.43 121.92) (xy 147.32 121.92)
+		)
+		(stroke
+			(width 0)
+			(type default)
+		)
+	)
+	(wire
+		(pts
+			(xy 138.43 107.95) (xy 147.32 107.95)
 		)
 		(stroke
@@
 	(bus
 		(pts
-			(xy 125.73 113.03) (xy 134.62 113.03)
+			(xy 138.43 111.76) (xy 147.32 111.76)
 		)
 		(stroke
@@
 	)
 	(sheet
-		(at 96.52 96.52)
+		(at 109.22 95.25)
 		(size 29.21 30.48)
 		(exclude_from_sim no)
@@
 		)
 		(property "Sheetname" "MCU"
-			(at 96.52 95.8084 0)
+			(at 109.22 94.5384 0)
 			(effects
 				(font
@@
 		)
 		(property "Sheetfile" "sch/mcu.kicad_sch"
-			(at 96.52 127.5846 0)
+			(at 109.22 126.3146 0)
 			(effects
 				(font
@@
 		)
 		(pin "LCD2_BL_EN" bidirectional
-			(at 125.73 123.19 0)
+			(at 138.43 121.92 0)
 			(effects
 				(font
@@
 		)
 		(pin "LCD2_CS" bidirectional
-			(at 125.73 115.57 0)
+			(at 138.43 114.3 0)
 			(effects
 				(font
@@
 		)
 		(pin "LCD_BL_EN" bidirectional
-			(at 125.73 102.87 0)
+			(at 138.43 101.6 0)
 			(effects
 				(font
@@
 		)
 		(pin "LCD{LCD}" bidirectional
-			(at 125.73 100.33 0)
+			(at 138.43 99.06 0)
 			(effects
 				(font
@@
 		)
 		(pin "OLED{I2C}" bidirectional
-			(at 125.73 106.68 0)
+			(at 138.43 105.41 0)
 			(effects
 				(font
@@
 		)
 		(pin "LCD2{I2C}" bidirectional
-			(at 125.73 113.03 0)
+			(at 138.43 111.76 0)
 			(effects
 				(font
@@
 		)
 		(pin "LCD2_RES" bidirectional
-			(at 125.73 118.11 0)
+			(at 138.43 116.84 0)
 			(effects
 				(font
@@
 		)
 		(pin "LCD2_A0" bidirectional
-			(at 125.73 120.65 0)
+			(at 138.43 119.38 0)
 			(effects
 				(font
@@
 		)
 		(pin "OLED_RST" bidirectional
-			(at 125.73 109.22 0)
+			(at 138.43 107.95 0)
 			(effects
 				(font
@@
 	)
 	(sheet
-		(at 134.62 96.52)
+		(at 147.32 95.25)
 		(size 29.21 30.48)
 		(exclude_from_sim no)
@@
 		)
 		(property "Sheetname" "OLED"
-			(at 134.62 95.8084 0)
+			(at 147.32 94.5384 0)
 			(effects
 				(font
@@
 		)
 		(property "Sheetfile" "sch/OLED.kicad_sch"
-			(at 134.62 127.5846 0)
+			(at 147.32 126.3146 0)
 			(effects
 				(font
@@
 		)
 		(pin "LCD{LCD}" bidirectional
-			(at 134.62 100.33 180)
+			(at 147.32 99.06 180)
 			(effects
 				(font
@@
 		)
 		(pin "LCD_BL_EN" bidirectional
-			(at 134.62 102.87 180)
+			(at 147.32 101.6 180)
 			(effects
 				(font
@@
 		)
 		(pin "LCD2{I2C}" bidirectional
-			(at 134.62 113.03 180)
+			(at 147.32 111.76 180)
 			(effects
 				(font
@@
 		)
 		(pin "LCD2_A0" bidirectional
-			(at 134.62 120.65 180)
+			(at 147.32 119.38 180)
 			(effects
 				(font
@@
 		)
 		(pin "LCD2_CS" bidirectional
-			(at 134.62 115.57 180)
+			(at 147.32 114.3 180)
 			(effects
 				(font
@@
 		)
 		(pin "LCD2_BL_EN" bidirectional
-			(at 134.62 123.19 180)
+			(at 147.32 121.92 180)
 			(effects
 				(font
@@
 		)
 		(pin "LCD2_RES" bidirectional
-			(at 134.62 118.11 180)
+			(at 147.32 116.84 180)
 			(effects
 				(font
@@
 		)
 		(pin "OLED{I2C}" bidirectional
-			(at 134.62 106.68 180)
+			(at 147.32 105.41 180)
 			(effects
 				(font
@@
 		)
 		(pin "OLED_RST" bidirectional
-			(at 134.62 109.22 180)
+			(at 147.32 107.95 180)
 			(effects
 				(font
@@
 	)
 	(sheet
-		(at 115.57 66.04)
+		(at 124.46 66.04)
 		(size 30.48 16.51)
 		(exclude_from_sim no)
@@
 		)
 		(property "Sheetname" "Power"
-			(at 115.57 65.3284 0)
+			(at 124.46 65.3284 0)
 			(effects
 				(font
@@
 		)
 		(property "Sheetfile" "sch/power.kicad_sch"
-			(at 115.57 83.1346 0)
-			(effects
-				(font
+			(at 124.46 83.1346 0)
+			(effects
+				(font
