File: Hardware/Tamagotchi-thing/Tamagotchi-thing.kicad_pcb (KiCad board)
At the start: 4 copper layers, 99 parts, among them J3 Conn_01x30, J5 Conn_01x30, J6 USB_C_Receptacle_USB2.0, J7 Conn_01x04, J8 Conn_01x04, Q1 BSS138, Q2 BSS138, Q3 AO3401A, Q4 AO3401A, Q5 FS8205A, SW1 SW_MEC_5E, SW2 SW_Push, SW3 RotaryEncoder_Switch_MP, SW4 SW_Push, SW5 SW_Push, SW6 SW_SPDT_321, U1 USBLC6-2P6, U2 STM32L073RBTx, U3 DW01A, U4 TPS63802DLAR, U5 TP4057, Y1 32768Hz - 12,5 pF

Commit message: Schematic and layout work
Parts:
- removed C1: 330nF/25V, Capacitor_SMD:C_0603_1608Metric
- removed C16, C17: 10nF, Capacitor_SMD:C_0603_1608Metric
- removed C2, C3: 2.2uF/5V, Capacitor_SMD:C_0603_1608Metric
- removed Q2: BSS138, Package_TO_SOT_SMD:SOT-23
- removed R23, R24, R5: 10k, Resistor_SMD:R_0603_1608Metric
- removed R29: 100k, Resistor_SMD:R_0603_1608Metric
- removed R30: 330, Resistor_SMD:R_0603_1608Metric
- removed R40, R41: 0, Resistor_SMD:R_0603_1608Metric
- removed SW3: RotaryEncoder_Switch_MP, TamagotchiThing:SW-SMD_SIQ-02FVS3
- added REF**: Tab, PCM_kikit:Tab, F.Cu at (164.3, 115.4)
- added REF**: Tab, PCM_kikit:Tab, F.Cu at (164.3, 68.4)
- added REF**: Tab, PCM_kikit:Tab, F.Cu at (135.6, 68.4)
- added REF**: Tab, PCM_kikit:Tab, F.Cu at (135.6, 115.4)
- BT1: footprint Connector_JST:JST_PH_S2B-PH-K_1x02_P2.00mm_Horizontal -> TamagotchiThing:Battery_Pads_4x4; moved to B.Cu
- C10, C13, C14, C15, C19, C20, C21, C23, C24, C5, C6, C7: footprint Capacitor_SMD:C_0603_1608Metric -> Capacitor_SMD:C_0402_1005Metric
- C11, C12, C4, C8, C9: footprint Capacitor_SMD:C_0603_1608Metric -> Capacitor_SMD:C_0402_1005Metric; moved to B.Cu
- J3, J6, JP1, LS1, U1: moved to B.Cu
- J5: footprint TamagotchiThing:sh1106-1.3inch-oled -> TamagotchiThing:sh1106-1.3inch-oled_1; moved to B.Cu
- R1, R11, R12, R13, R14, R16, R17, R18, R19, R2, R21, R22, R25, R26, R27, R28, R3, R31, R32, R34, R35, R36, R37, R38, R39, R4, R42, R6, R7: footprint Resistor_SMD:R_0603_1608Metric -> Resistor_SMD:R_0402_1005Metric
- R10, R8, R9: footprint Resistor_SMD:R_0603_1608Metric -> Capacitor_SMD:C_0402_1005Metric
- R15: footprint Resistor_SMD:R_0603_1608Metric -> Resistor_SMD:R_0402_1005Metric; moved to B.Cu
- R33: value 10k -> 100k; footprint Resistor_SMD:R_0603_1608Metric -> Resistor_SMD:R_0402_1005Metric
- moved C15 121.6 mm to (207.2, 91.2), turned to 90 degrees
- moved SW1 116.7 mm to (203.7, 91.3)
- moved R12 114.1 mm to (203.7, 93.9)
- moved R11 112.5 mm to (201.7, 93.9)
- moved R1 104.8 mm to (187.2, 76.5)
- moved R2 104.8 mm to (187.2, 79.0)
- moved Q1 100.4 mm to (190.6, 77.7)
- moved JP1 93.7 mm to (178.2, 70.7), turned to 180 degrees
- moved C12 92.5 mm to (159.3, 76.4)
- moved R15 88.4 mm to (178.2, 72.7)
- moved C6 88.0 mm to (149.8, 77.0), turned to 180 degrees
- moved C5 87.7 mm to (151.7, 77.0), turned to 180 degrees
- moved C10 86.1 mm to (155.7, 76.8), turned to -90 degrees
- moved C9 86.1 mm to (157.4, 76.4)
- moved C4 84.7 mm to (153.2, 80.9)
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Connections:
- U5 pad 2: Net-(U5-GND) -> GND
Routing:
- net GND: track 0.00 -> 55.5 mm, vias 0 -> 46
- net Net-(SW6-A): track 0.00 -> 25.0 mm, vias 0 -> 7
- net 3V3: track 0.00 -> 20.7 mm, vias 0 -> 18
- net Net-(D3-K2): track 0.00 -> 14.4 mm, vias 0 -> 1
- net Net-(D3-K1): track 0.00 -> 13.1 mm, vias 0 -> 1
- net VBUS: track 0.00 -> 9.64 mm, vias 0 -> 12
- net 3V3A: track 0.00 -> 6.32 mm
- net /MCU/OSC_32_OUT: track 0.00 -> 5.46 mm
- net /MCU/OSC_32_IN: track 0.00 -> 5.46 mm
- net Net-(U3-CS): track 0.00 -> 4.11 mm
- net Net-(U4-FB): track 0.00 -> 3.98 mm
- net GND_BAT: track 0.00 -> 3.91 mm, vias 0 -> 12
- net Net-(U4-L1): track 0.00 -> 3.02 mm
- net Net-(U4-L2): track 0.00 -> 3.02 mm
- net Net-(J5-Pin_5): track 0.00 -> 2.86 mm
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- added copper zone on F.Cu, net 3V3
- added copper zone on In2.Cu, net 3V3
- added copper zone on B.Cu, net GND
- added copper zone on F.Cu, net GND
- added copper zone on In1.Cu, net GND
- added copper zone on B.Cu, net GND_BAT
- added copper zone on F.Cu, net GND_BAT
- added copper zone on F.Cu, net Net-(D1-K)
- added copper zone on F.Cu, net Net-(Q4-G)
- added copper zone on F.Cu, net Net-(SW6-A)
- added copper zone on B.Cu, net VBAT
- added copper zone on F.Cu, net VBAT
- added copper zone on F.Cu, net VBUS
- added copper zone on In2.Cu, net VBUS
Other:
- board outline added: 42.5 x 47 mm

Commit message: Schematic and Layout work
Parts:
- removed SW1: SW_MEC_5E, TamagotchiThing:SW_SKRPACE010
- added C28: 100nF, Capacitor_SMD:C_0402_1005Metric, B.Cu at (163.8, 78.5)
- added J1: Conn_01x14, Resistor_SMD:R_1210_3225Metric, B.Cu at (133.5, 93.8)
- Q1, R1, R2, R3, R4, R6, R8, R9: moved to B.Cu
- R20: footprint Resistor_SMD:R_0603_1608Metric -> Resistor_SMD:R_0402_1005Metric; moved to B.Cu
- moved R4 107.5 mm to (153.2, 83.0), turned to 180 degrees
- moved R9 105.6 mm to (157.6, 85.1)
- moved R8 105.5 mm to (157.8, 83.0)
- moved R3 104.8 mm to (152.7, 85.0), turned to 180 degrees
- moved C18 95.5 mm to (148.2, 91.8), turned to 180 degrees
- moved R31 93.9 mm to (157.4, 100.0), turned to 180 degrees
- moved R32 93.7 mm to (157.4, 101.0)
- moved R20 87.8 mm to (148.5, 79.4)
- moved R17 87.7 mm to (143.0, 79.4), turned to 180 degrees
- moved R16 87.4 mm to (143.0, 78.4)
- moved R27 86.8 mm to (147.8, 100.3), turned to 180 degrees
- moved R28 86.4 mm to (147.8, 101.3)
- moved R21 79.5 mm to (138.2, 100.2), turned to 180 degrees
- moved R22 79.2 mm to (138.2, 101.2)
- moved C15 63.6 mm to (143.6, 89.8)
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Connections:
- D3 pad 2: Net-(D3-A1) -> Net-(D3-K2)
- D3 pad 3: Net-(D3-K2) -> Net-(D3-A1)
- U2 pad 16: unconnected-(U2-PA2-Pad16) -> /MCU/SW_LEFT
- U2 pad 17: unconnected-(U2-PA3-Pad17) -> /MCU/SW_CENTER
- U2 pad 28: unconnected-(U2-PB2-Pad28) -> /MCU/SW_RIGHT
Routing:
- net 3V3: track 20.7 -> 101.6 mm, vias 18 -> 34
- net /MCU/UART_TX: track 0.00 -> 26.4 mm, vias 0 -> 2
- net /MCU/UART_RX: track 0.00 -> 24.9 mm, vias 0 -> 2
- net /MCU/OLED.SCL: track 1.78 -> 25.8 mm, vias 1 -> 3
- net /MCU/VBAT_SENSE: track 0.00 -> 24.0 mm, vias 0 -> 2
- net /MCU/OLED.SDA: track 2.46 -> 25.7 mm, vias 1 -> 3
- net /MCU/SWCLK: track 0.00 -> 22.0 mm, vias 0 -> 1
- net /MCU/OLED_RST: track 1.75 -> 23.7 mm, vias 1 -> 2
- net /MCU/SW_LEFT: track 0.00 -> 20.2 mm
- net /MCU/SPK: track 0.00 -> 19.9 mm, vias 0 -> 2
- net Net-(J1-Pin_2): track 0.00 -> 19.7 mm, vias 0 -> 2
- net /MCU/LCD2_CS: track 2.18 -> 21.0 mm
- net VBUS: track 9.64 -> 28.1 mm, vias 12 -> 13
- net /MCU/SWDIO: track 0.00 -> 17.7 mm, vias 0 -> 1
- net /MCU/LCD2_BL_EN: track 0.00 -> 17.0 mm, vias 0 -> 2
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- added copper zone on In2.Cu, net GND

Commit message: Schematic and Layout work. DRC cleanup
Parts:
- moved R13 2.86 mm to (164.2, 72.2)
- moved R20 0.88 mm to (148.6, 80.3)
- moved C28 0.55 mm to (164.4, 78.5)
- moved J6 0.55 mm to (166.1, 72.1)
- moved U1 0.55 mm to (166.2, 79.9)
- moved R14 0.40 mm to (164.2, 73.3)
- moved LS1 0.33 mm to (134.1, 74.5)
Routing:
- net Net-(J6-CC2): track 0.00 -> 6.20 mm, vias 0 -> 1
- net /MCU/USB_D_N: track 12.0 -> 7.68 mm
- net Net-(J6-CC1): track 0.00 -> 2.63 mm, vias 0 -> 1
- net 3V3: track 101.6 -> 104.3 mm
- net /MCU/USB_D_P: track 9.33 -> 6.89 mm
- net GND: track 70.8 -> 71.6 mm, vias 58 -> 57
Other:
- outline, holes or cut-outs redrawn
- board text added: "3V3"
- board text added: "Afonso Muralha 2k25"
- board text added: "GND"
- board text added: "RX"
- board text added: "SWCLK"
- board text added: "SWDIO"
- board text added: "TX"

Commit message: Final touches. Exported production files
Parts:
- C10, C11, C12, C7, C9: value 2.2u -> 2.2uF
- C25, C27: value 10u -> 10uF
- C26: value 22u -> 22uF
- C8: value 4.7u -> 4.7uF

Commit message: Minor fixes. Added via stitching. BOM adjustments. Sent to production
Routing:
- net GND: vias 57 -> 147
