File: Hardware/Tamagotchi-thing/sch/mcu.kicad_sch (KiCad schematic)
At the start: 22 parts, among them J6 USB_C_Receptacle_USB2.0, SW1 SW_Push, SW2 SW_Push, SW3 SW_Push, SW4 SW_MEC_5E, U1 USBLC6-2P6, U4 STM32L073RBTx, Y1 32768Hz - 12,5 pF

Commit message: schematic work
Parts:
- added J2, J3: Conn_01x04, Connector_PinHeader_2.54mm:PinHeader_1x04_P2.54mm_Horizontal, symbol Connector_Generic:Conn_01x04
- added R27, R28, R29, R30: 330, symbol Device:R_Small_US
- added R31, R32: 100k, symbol Device:R_Small_US
- R10: symbol Device:R_Small -> Device:R_Small_US; LCSC C11702 -> (none)
- R9: symbol Device:R_Small -> Device:R_Small_US; LCSC C25076 -> (none)
Connections:
- net 3V3: now also J2.1 (Pin_1), J3.1 (Pin_1)
- net GND: now also J2.4 (Pin_4), J3.4 (Pin_4), R32.2
- net LCD_BL_EN: now also U4.27 (PB1)
- net RST: now also R30.2; no longer C6.1, R19.2, SW4.3 (K), SW4.4 (A)
- net SW_CENTER: now also R28.1; no longer R3.1, SW2.1
- net SW_LEFT: now also R27.1; no longer R2.1, SW1.1
- net SW_RIGHT: now also R29.1; no longer R14.1, SW3.1
- net VBUS_SENSE: now also U4.61 (PB8)
- net VBAT_SENSE: now reaches U4.26 (PB0)
- net VBAT_SENSE: now also R31.2, R32.1
- net SWDIO: now reaches U4.46 (PA13)
- net SWDIO: now also J2.2 (Pin_2)
- net SWCLK: now reaches U4.49 (PA14)
- net SWCLK: now also J2.3 (Pin_3)
- net VBUS_IN renamed VBUS
- new net: R14.1, R29.2, SW3.1
- new net: C6.1, R19.2, R30.1, SW4.3 (K), SW4.4 (A)
- new net: R2.1, R27.2, SW1.1
- new net: R28.2, R3.1, SW2.1
- new net UART_RX: J3.3 (Pin_3)
- new net UART_TX: J3.2 (Pin_2)
- new net VBAT: R31.1
Other:
- moved on the sheet: R14, R3, SW2, SW3

Commit message: Schematic work
Parts:
- added C16: 1uF, Capacitor_SMD:C_0603_1608Metric, symbol Device:C_Small
- added C17, C21, C22, C23: 10nF, Capacitor_SMD:C_0402_1005Metric, symbol Device:C_Small
- added C18, C19, C20: 100nF, Capacitor_SMD:C_0603_1608Metric, symbol Device:C_Small
- added JP1: SolderJumper_2_Open, Jumper:SolderJumper-2_P1.3mm_Open_Pad1.0x1.5mm, symbol Jumper:SolderJumper_2_Open
- added L2: 39nH, Inductor_SMD:L_0402_1005Metric, symbol Device:L_Small
- added R33: 0, symbol Device:R_Small_US
- added R34: 100k, Resistor_SMD:R_0603_1608Metric, symbol Device:R_Small_US
- added R35, R36: 10k, Resistor_SMD:R_0402_1005Metric, symbol Device:R_Small_US
- added R37: 330, symbol Device:R_Small_US
- added R38: 100k, symbol Device:R_Small_US
- added SW5: RotaryEncoder_Switch_MP, TamagotchiThing:SW-SMD_SIQ-02FVS3, symbol Device:RotaryEncoder_Switch_MP
- SW1, SW2, SW3: footprint (none) -> TamagotchiThing:Kailh_mouse_button; now left out of the parts list
Connections:
- net 3V3: now also U4.19 (VDD), U4.32 (VDD), U4.48 (VDD_USB), U4.64 (VDD), C18.1, C19.1, C20.1, C21.1, JP1.1 (A), L2.1, R33.1, R38.1
- net GND: now also U4.12 (VSSA), U4.18 (VSS), U4.31 (VSS), U4.47 (VSS), U4.63 (VSS), C16.2, C17.2, C18.2, C19.2, C20.2, C21.2, C22.2, C23.2, R34.2, SW5.C, SW5.MP
- net UART_RX: now also U4.15 (PA1)
- net UART_TX: now also U4.14 (PA0)
- net at U4.1 (VLCD): now also R33.2
- net LCD2_A0: now reaches U4.10 (PC2)
- net LCD2_RES: now reaches U4.11 (PC3)
- net 3V3A: now reaches U4.13 (VDDA)
- net 3V3A: now also C16.1, C17.1, L2.2
- net LCD2_CS: now reaches U4.24 (PC4)
- net OLED_RST: now reaches U4.25 (PC5)
- net LCD2_BL_EN: now reaches U4.57 (PB5)
- net BOOT0: now reaches U4.60 (BOOT0)
- net BOOT0: now also JP1.2 (B), R34.1
- net LCD2.SCL: now reaches U4.8 (PC0)
- net LCD2.SDA: now reaches U4.9 (PC1)
- new net: R35.1, SW5.A
- new net: R36.2, SW5.B
- new net: R37.2, R38.2, SW5.S
- new net ENC_A: C22.1, R35.2
- new net ENC_B: C23.1, R36.1
- new net ENC_S: R37.1
Other:
- moved on the sheet: C3, C6, J2, J3, LS1, R10, R19, R30, R9, SW4, U4, Y1

Commit message: Schematic and layout work
Parts:
- C13, C14: renamed from C3; footprint Capacitor_SMD:C_0402_1005Metric -> Capacitor_SMD:C_0603_1608Metric
- C16: renamed from C22; footprint Capacitor_SMD:C_0402_1005Metric -> Capacitor_SMD:C_0603_1608Metric
- C17: renamed from C23; footprint Capacitor_SMD:C_0402_1005Metric -> Capacitor_SMD:C_0603_1608Metric
- C18: renamed from C21; footprint Capacitor_SMD:C_0402_1005Metric -> Capacitor_SMD:C_0603_1608Metric
- C23: renamed from C17; footprint Capacitor_SMD:C_0402_1005Metric -> Capacitor_SMD:C_0603_1608Metric
- R12: renamed from R30; footprint (none) -> Resistor_SMD:R_0603_1608Metric
- R16: renamed from R17; footprint (none) -> Resistor_SMD:R_0603_1608Metric
- R17: renamed from R18; footprint (none) -> Resistor_SMD:R_0603_1608Metric
- R18: renamed from R31; footprint (none) -> Resistor_SMD:R_0603_1608Metric
- R19: renamed from R32; footprint (none) -> Resistor_SMD:R_0603_1608Metric
- R20: renamed from R33; footprint (none) -> Resistor_SMD:R_0603_1608Metric
- R21: renamed from R27; footprint (none) -> Resistor_SMD:R_0603_1608Metric
- R22: renamed from R2; footprint (none) -> Resistor_SMD:R_0603_1608Metric
- R23: renamed from R35; footprint Resistor_SMD:R_0402_1005Metric -> Resistor_SMD:R_0603_1608Metric
- R24: renamed from R36; footprint Resistor_SMD:R_0402_1005Metric -> Resistor_SMD:R_0603_1608Metric
- R25: renamed from R9; footprint Resistor_SMD:R_0402_1005Metric -> Resistor_SMD:R_0603_1608Metric
- R26: renamed from R10; footprint Resistor_SMD:R_0402_1005Metric -> Resistor_SMD:R_0603_1608Metric
- R27: renamed from R28; footprint (none) -> Resistor_SMD:R_0603_1608Metric
- R28: renamed from R3; footprint (none) -> Resistor_SMD:R_0603_1608Metric
- R29: renamed from R38; footprint (none) -> Resistor_SMD:R_0603_1608Metric
- R30: renamed from R37; footprint (none) -> Resistor_SMD:R_0603_1608Metric
- R31: renamed from R29; footprint (none) -> Resistor_SMD:R_0603_1608Metric
- R32: renamed from R14; footprint (none) -> Resistor_SMD:R_0603_1608Metric
- SW1: renamed from SW4; footprint Bongo-Cat-Fidget-Toy:SW_SKRPACE010 -> TamagotchiThing:SW_SKRPACE010
- Y1: footprint (none) -> Crystal:Crystal_SMD_3215-2Pin_3.2x1.5mm; LCSC (none) -> C32346
- renumbered C6 to C15, C18 to C19, C19 to C20, C20 to C21, C16 to C22, J2 to J7, J3 to J8, L2 to L1, R19 to R11, R15 to R13, R16 to R14, R34 to R15, SW1 to SW2, SW5 to SW3, SW2 to SW4, SW3 to SW5, U4 to U2
Other:
- company: (none) -> Afonso Muralha
- title: (none) -> MCU
- moved on the sheet: C13, C14, Y1

Commit message: Schematic and layout work
Parts:
- C13, C14, C15, C19, C20, C21, C23: footprint Capacitor_SMD:C_0603_1608Metric -> Capacitor_SMD:C_0402_1005Metric
- C16, C17: footprint Capacitor_SMD:C_0603_1608Metric -> Capacitor_SMD:C_0402_1005Metric; now not fitted; now left out of the parts list
- R11, R12, R13, R14, R16, R17, R18, R19, R21, R22, R25, R26, R27, R28, R31, R32: footprint Resistor_SMD:R_0603_1608Metric -> Resistor_SMD:R_0402_1005Metric
- R15: footprint Resistor_SMD:R_0603_1608Metric -> Resistor_SMD:R_0402_1005Metric; LCSC C25803 -> (none)
- R23, R24, R29, R30, SW3: now not fitted; now left out of the parts list
Changed lines of the file:
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@@
 			)
 		)
-		(property "Footprint" "Capacitor_SMD:C_0603_1608Metric"
+		(property "Footprint" "Capacitor_SMD:C_0402_1005Metric"
 			(at 62.23 58.42 0)
 			(effects
@@
 			)
 		)
-		(property "Footprint" "Resistor_SMD:R_0603_1608Metric"
+		(property "Footprint" "Resistor_SMD:R_0402_1005Metric"
 			(at 223.52 100.33 0)
 			(effects
@@
 			)
 		)
-		(property "Footprint" "Resistor_SMD:R_0603_1608Metric"
+		(property "Footprint" "Resistor_SMD:R_0402_1005Metric"
 			(at 229.87 104.14 0)
 			(effects
@@
 			)
 		)
-		(property "Footprint" "Capacitor_SMD:C_0603_1608Metric"
+		(property "Footprint" "Capacitor_SMD:C_0402_1005Metric"
 			(at 269.24 45.72 0)
 			(effects
@@
 		(unit 1)
 		(exclude_from_sim no)
-		(in_bom yes)
-		(on_board yes)
-		(dnp no)
+		(in_bom no)
+		(on_board no)
+		(dnp yes)
 		(fields_autoplaced yes)
 		(property "Reference" "SW3"
@@
 		(unit 1)
 		(exclude_from_sim no)
-		(in_bom yes)
-		(on_board yes)
-		(dnp no)
+		(in_bom no)
+		(on_board no)
+		(dnp yes)
 		(property "Reference" "R23"
 			(at 215.9 63.3984 90)
@@
 			)
 		)
-		(property "Footprint" "Resistor_SMD:R_0603_1608Metric"
+		(property "Footprint" "Resistor_SMD:R_0402_1005Metric"
 			(at 64.77 153.67 0)
 			(effects
@@
 			)
 		)
-		(property "Footprint" "Resistor_SMD:R_0603_1608Metric"
+		(property "Footprint" "Resistor_SMD:R_0402_1005Metric"
 			(at 104.14 52.07 0)
 			(effects
@@
 			)
 		)
-		(property "LCSC" "C25803"
+		(property "LCSC" ""
 			(at 104.14 52.07 0)
 			(effects
@@
 			)
 		)
-		(property "Footprint" "Resistor_SMD:R_0603_1608Metric"
+		(property "Footprint" "Resistor_SMD:R_0402_1005Metric"
 			(at 116.84 181.61 0)
 			(effects
@@
 			)
 		)
-		(property "Footprint" "Resistor_SMD:R_0603_1608Metric"
+		(property "Footprint" "Resistor_SMD:R_0402_1005Metric"
 			(at 259.08 139.7 0)
 			(effects
@@
 			)
 		)
-		(property "Footprint" "Resistor_SMD:R_0603_1608Metric"
+		(property "Footprint" "Resistor_SMD:R_0402_1005Metric"
 			(at 264.16 143.51 0)
 			(effects
@@
 			)
 		)
-		(property "Footprint" "Resistor_SMD:R_0603_1608Metric"
+		(property "Footprint" "Resistor_SMD:R_0402_1005Metric"
 			(at 46.99 83.82 0)
 			(effects
@@
 			)
 		)
-		(property "Footprint" "Resistor_SMD:R_0603_1608Metric"
+		(property "Footprint" "Resistor_SMD:R_0402_1005Metric"
 			(at 138.43 181.61 0)
 			(effects
@@
 		(unit 1)
 		(exclude_from_sim no)
-		(in_bom yes)
-		(on_board yes)
-		(dnp no)
+		(in_bom no)
+		(on_board no)
+		(dnp yes)
 		(property "Reference" "R30"
 			(at 256.286 71.12 90)
@@
 			)
 		)
-		(property "Footprint" "Resistor_SMD:R_0603_1608Metric"
+		(property "Footprint" "Resistor_SMD:R_0402_1005Metric"
 			(at 34.29 78.74 0)
 			(effects
@@
 			)
 		)
-		(property "Footprint" "Resistor_SMD:R_0603_1608Metric"
+		(property "Footprint" "Resistor_SMD:R_0402_1005Metric"
 			(at 233.68 139.7 0)
 			(effects
@@
 		(unit 1)
 		(exclude_from_sim no)
-		(in_bom yes)
-		(on_board yes)
-		(dnp no)
+		(in_bom no)
+		(on_board no)
+		(dnp yes)
 		(fields_autoplaced yes)
 		(property "Reference" "R29"
@@
 			)
 		)
-		(property "Footprint" "Capacitor_SMD:C_0603_1608Metric"
+		(property "Footprint" "Capacitor_SMD:C_0402_1005Metric"
 			(at 223.52 45.72 0)
 			(effects
@@
 			)
 		)
-		(property "Footprint" "Resistor_SMD:R_0603_1608Metric"
+		(property "Footprint" "Resistor_SMD:R_0402_1005Metric"
 			(at 210.82 143.51 0)
 			(effects
@@
 			)
 		)
-		(property "Footprint" "Resistor_SMD:R_0603_1608Metric"
+		(property "Footprint" "Resistor_SMD:R_0402_1005Metric"
 			(at 205.74 139.7 0)
 			(effects
@@
 			)
 		)
-		(property "Footprint" "Capacitor_SMD:C_0603_1608Metric"
+		(property "Footprint" "Capacitor_SMD:C_0402_1005Metric"
 			(at 246.38 45.72 0)
 			(effects
@@
 		(unit 1)
 		(exclude_from_sim no)
-		(in_bom yes)
-		(on_board yes)
-		(dnp no)
+		(in_bom no)
+		(on_board no)
+		(dnp yes)
 		(property "Reference" "R24"
 			(at 215.9 84.9884 90)
@@
 			)
 		)
-		(property "Footprint" "Resistor_SMD:R_0603_1608Metric"
+		(property "Footprint" "Resistor_SMD:R_0402_1005Metric"
 			(at 138.43 173.99 0)
 			(effects
@@
 		(unit 1)
 		(exclude_from_sim no)
-		(in_bom yes)
-		(on_board yes)
-		(dnp no)
+		(in_bom no)
+		(on_board no)
+		(dnp yes)
 		(property "Reference" "C17"
 			(at 208.4832 82.6516 0)
@@
 			)
 		)
-		(property "Footprint" "Capacitor_SMD:C_0603_1608Metric"
+		(property "Footprint" "Capacitor_SMD:C_0402_1005Metric"
 			(at 210.82 83.82 0)
 			(effects
@@
 			)
 		)
-		(property "Footprint" "Capacitor_SMD:C_0603_1608Metric"
+		(property "Footprint" "Capacitor_SMD:C_0402_1005Metric"
 			(at 52.07 58.42 0)
 			(effects
@@
 			)
 		)
-		(property "Footprint" "Capacitor_SMD:C_0603_1608Metric"
+		(property "Footprint" "Capacitor_SMD:C_0402_1005Metric"
 			(at 234.95 45.72 0)
 			(effects
@@
 			)
 		)
-		(property "Footprint" "Resistor_SMD:R_0603_1608Metric"
+		(property "Footprint" "Resistor_SMD:R_0402_1005Metric"
 			(at 238.76 143.51 0)
 			(effects
@@
 			)
 		)
-		(property "Footprint" "Resistor_SMD:R_0603_1608Metric"
+		(property "Footprint" "Resistor_SMD:R_0402_1005Metric"
 			(at 116.84 173.99 0)
 			(effects
@@
 		(unit 1)
 		(exclude_from_sim no)
-		(in_bom yes)
-		(on_board yes)
-		(dnp no)
+		(in_bom no)
+		(on_board no)
+		(dnp yes)
 		(property "Reference" "C16"
 			(at 208.4832 61.0616 0)
@@
 			)
 		)
-		(property "Footprint" "Capacitor_SMD:C_0603_1608Metric"
+		(property "Footprint" "Capacitor_SMD:C_0402_1005Metric"
 			(at 210.82 62.23 0)
 			(effects
@@
 			)
 		)
-		(property "Footprint" "Resistor_SMD:R_0603_1608Metric"
+		(property "Footprint" "Resistor_SMD:R_0402_1005Metric"
 			(at 73.66 153.67 0)
 			(effects
@@
 			)
 		)
-		(property "Footprint" "Capacitor_SMD:C_0603_1608Metric"
+		(property "Footprint" "Capacitor_SMD:C_0402_1005Metric"
 			(at 41.91 88.9 0)
 			(effects

Commit message: Schematic and Layout work
Parts:
- removed SW1: SW_MEC_5E, TamagotchiThing:SW_SKRPACE010, symbol Switch:SW_MEC_5E
- added C28: 100nF, Capacitor_SMD:C_0402_1005Metric, symbol Device:C_Small
- R20: footprint Resistor_SMD:R_0603_1608Metric -> Resistor_SMD:R_0402_1005Metric
Connections:
- net GND: now also C28.2
- net SW_CENTER: now also U2.17 (PA3)
- net SW_LEFT: now also U2.16 (PA2)
- net SW_RIGHT: now also U2.28 (PB2)
- net VBUS: now also C28.1
Other:
- moved on the sheet: C15, R12

Commit message: Final touches. Exported production files
Parts:
- C15, C19, C20, C21, C28: LCSC C30926 -> C2180552
- R12, R21, R27, R30, R31: LCSC (none) -> C105875
- R15, R16, R17, R18, R19, R22, R28, R29, R32: LCSC (none) -> C60491
- R20: LCSC (none) -> C106231
- R23, R24: LCSC (none) -> C60490
- R25: LCSC (none) -> C106232
- R26: LCSC (none) -> C106235
- U2: LCSC (none) -> C2917159
Changed lines of the file:
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@@
 			)
 		)
-		(property "LCSC" ""
+		(property "LCSC" "C106232"
 			(at 223.52 100.33 0)
 			(effects
@@
 			)
 		)
-		(property "LCSC" ""
+		(property "LCSC" "C106235"
 			(at 229.87 104.14 0)
 			(effects
@@
 			)
 		)
-		(property "LCSC" ""
+		(property "LCSC" "C60490"
 			(at 215.9 58.42 0)
 			(effects
@@
 			)
 		)
-		(property "LCSC" ""
+		(property "LCSC" "C60491"
 			(at 104.14 52.07 0)
 			(effects
@@
 			)
 		)
+		(property "LCSC" "C60491"
+			(at 116.84 181.61 0)
+			(effects
+				(font
+					(size 1.27 1.27)
+				)
+				(hide yes)
+			)
+		)
 		(pin "2"
 		)
@@
 			)
 		)
+		(property "LCSC" "C105875"
+			(at 259.08 139.7 90)
+			(effects
+				(font
+					(size 1.27 1.27)
+				)
+				(hide yes)
+			)
+		)
 		(pin "2"
 		)
@@
 			)
 		)
+		(property "LCSC" "C60491"
+			(at 264.16 143.51 0)
+			(effects
+				(font
+					(size 1.27 1.27)
+				)
+				(hide yes)
+			)
+		)
 		(pin "2"
 		)
@@
 			)
 		)
+		(property "LCSC" "C105875"
+			(at 39.37 83.82 90)
+			(effects
+				(font
+					(size 1.27 1.27)
+				)
+				(hide yes)
+			)
+		)
 		(pin "2"
 		)
@@
 			)
 		)
+		(property "LCSC" "C60491"
+			(at 138.43 181.61 0)
+			(effects
+				(font
+					(size 1.27 1.27)
+				)
+				(hide yes)
+			)
+		)
 		(pin "2"
 		)
@@
 			)
 		)
+		(property "LCSC" "C105875"
+			(at 252.73 72.39 90)
+			(effects
+				(font
+					(size 1.27 1.27)
+				)
+				(hide yes)
+			)
+		)
 		(pin "2"
 		)
@@
 			)
 		)
+		(property "LCSC" "C105875"
+			(at 233.68 139.7 90)
+			(effects
+				(font
+					(size 1.27 1.27)
+				)
+				(hide yes)
+			)
+		)
 		(pin "2"
 		)
@@
 			)
 		)
+		(property "LCSC" "C60491"
+			(at 245.11 67.31 0)
+			(effects
+				(font
+					(size 1.27 1.27)
+				)
+				(hide yes)
+			)
+		)
 		(pin "2"
 		)
@@
 			)
 		)
+		(property "LCSC" "C106231"
+			(at 144.78 31.75 0)
+			(effects
+				(font
+					(size 1.27 1.27)
+				)
+				(hide yes)
+			)
+		)
 		(pin "1"
 		)
@@
 			)
 		)
-		(property "LCSC" "C30926"
+		(property "LCSC" "C2180552"
 			(at 223.52 45.72 0)
 			(effects
@@
 			)
 		)
+		(property "LCSC" "C60491"
+			(at 210.82 143.51 0)
+			(effects
+				(font
+					(size 1.27 1.27)
+				)
+				(hide yes)
+			)
+		)
 		(pin "2"
 		)
@@
 			)
 		)
+		(property "LCSC" "C105875"
+			(at 205.74 139.7 90)
+			(effects
+				(font
+					(size 1.27 1.27)
+				)
+				(hide yes)
+			)
+		)
 		(pin "2"
 		)
@@
 			)
 		)
-		(property "LCSC" "C30926"
+		(property "LCSC" "C2180552"
 			(at 246.38 45.72 0)
 			(effects
@@
 			)
 		)
-		(property "LCSC" ""
+		(property "LCSC" "C60490"
 			(at 215.9 80.01 0)
 			(effects
@@
 			)
 		)
+		(property "LCSC" "C60491"
+			(at 138.43 173.99 0)
+			(effects
+				(font
+					(size 1.27 1.27)
+				)
+				(hide yes)
+			)
+		)
 		(pin "2"
 		)
@@
 			)
 		)
-		(property "LCSC" "C30926"
+		(property "LCSC" "C2180552"
 			(at 57.15 182.88 0)
 			(effects
@@
 			)
 		)
-		(property "LCSC" "C30926"
+		(property "LCSC" "C2180552"
 			(at 234.95 45.72 0)
 			(effects
@@
 			)
 		)
+		(property "LCSC" "C60491"
+			(at 238.76 143.51 0)
+			(effects
+				(font
+					(size 1.27 1.27)
+				)
+				(hide yes)
+			)
+		)
 		(pin "2"
 		)
@@
 			)
 		)
+		(property "LCSC" "C60491"
+			(at 116.84 173.99 0)
+			(effects
+				(font
+					(size 1.27 1.27)
+				)
+				(hide yes)
+			)
+		)
 		(pin "2"
 		)
@@
 			)
 		)
-		(property "LCSC" "C30926"
+		(property "LCSC" "C2180552"
 			(at 34.29 88.9 0)
 			(effects
@@
 			(at 137.16 83.82 0)
 			(effects
+				(font
+					(size 1.27 1.27)
+				)
+				(hide yes)
+			)
+		)
+		(property "LCSC" "C2917159"
+			(at 137.16 83.82 0)
+			(effects
