File: Hardware/Tamagotchi-thing/sch/power.kicad_sch (KiCad schematic)
At the start: 25 parts, among them Q1 AO3401A, Q3 FS8205A, Q4 AO3401A, U101 TPS63802DLAR, U3 DW01A, U6 TP4057

Commit message: Schematic work
Parts:
- added SW6: SW_SPDT_321, Bongo-Cat-Fidget-Toy:SW-SMD_SK-3245S-L1-A-1, symbol Switch:SW_SPDT_321
Connections:
- net at C1.1, U101.1 (EN), U101.10 (VIN): now also SW6.3 (A); no longer D1.1 (K), D3.1 (K), Q1.2 (S)
- net at D2.2 (A1), R24.2: now also D2.4 (A2); no longer D2.1 (A1)
- net at U6.1 (~{CHRG}): now also D2.1 (K1); no longer D2.3 (K1)
- net at U6.5 (STDBY): now also D2.3 (K2); no longer D2.4 (K2)
- new net: D1.1 (K), D3.1 (K), Q1.2 (S), SW6.2 (B)
- no-connect marks 1 -> 2
Other:
- moved on the sheet: C1, C2, D1, D3, L102, Q1, R4, R5, R6, U101

Commit message: Schematic and layout work
Parts:
- BT1: renamed from BT2; footprint Bongo-Cat-Fidget-Toy:BAT-TH_CR2032-BS-6-1 -> Connector_JST:JST_PH_S2B-PH-K_1x02_P2.00mm_Horizontal
- C24: renamed from C7; footprint (none) -> Capacitor_SMD:C_0603_1608Metric
- D3: renamed from D2; footprint (none) -> TamagotchiThing:LED-SMD_4P-L1.6-W1.5-TL-1
- R33: renamed from R5; value 10k -> 100k; LCSC C103199 -> (none)
- R34: renamed from R26; footprint (none) -> Resistor_SMD:R_0603_1608Metric
- R35: renamed from R20; footprint (none) -> Resistor_SMD:R_0603_1608Metric
- R36: renamed from R21; footprint (none) -> Resistor_SMD:R_0603_1608Metric
- R39: renamed from R24; footprint (none) -> Resistor_SMD:R_0603_1608Metric
- R40: renamed from R22; footprint (none) -> Resistor_SMD:R_0603_1608Metric; now not fitted
- R41: renamed from R23; footprint (none) -> Resistor_SMD:R_0603_1608Metric
- R42: renamed from R25; footprint (none) -> Resistor_SMD:R_0603_1608Metric
- SW6: footprint Bongo-Cat-Fidget-Toy:SW-SMD_SK-3245S-L1-A-1 -> TamagotchiThing:SW-SMD_SK-3245S-L1-A-1
- U4: renamed from U101; footprint Bongo-Cat-Fidget-Toy:VREG_TPS63802DLAR -> TamagotchiThing:VREG_TPS63802DLAR
- renumbered C1 to C25, C2 to C26, C14 to C27, D3 to D2, L102 to L2, Q1 to Q3, Q3 to Q5, R6 to R37, R4 to R38, U6 to U5
Connections:
- net GND: now also Q5.3 (S2); no longer Q5.1 (D1)
- net GND_BAT: now also Q5.1 (D1); no longer Q5.3 (S2)
- net at Q4.1 (G), U3.1 (OD): now also Q5.6 (G1); no longer Q5.4 (G2)
- net at U3.3 (OC): now also Q5.4 (G2); no longer Q5.6 (G1)
Other:
- company: (none) -> Afonso Muralha
- title: (none) -> Power
- moved on the sheet: Q5

Commit message: Schematic and layout work
Parts:
- removed R40, R41: 0, Resistor_SMD:R_0603_1608Metric, symbol Device:R_Small_US
- BT1: footprint Connector_JST:JST_PH_S2B-PH-K_1x02_P2.00mm_Horizontal -> TamagotchiThing:Battery_Pads_4x4
- C24: footprint Capacitor_SMD:C_0603_1608Metric -> Capacitor_SMD:C_0402_1005Metric
- R33, R34, R35, R36, R37, R38, R39, R42: footprint Resistor_SMD:R_0603_1608Metric -> Resistor_SMD:R_0402_1005Metric
Connections:
- net GND: now also U5.2 (GND)
Other:
- moved on the sheet: R42

Commit message: Schematic and Layout work
Parts:
- removed D3: LED_Dual_KKA, TamagotchiThing:LED-SMD_4P-L1.6-W1.5-TL-1, symbol Device:LED_Dual_AAKK
- added D3: LED_Dual_KKA, TamagotchiThing:LED-SMD_4P-L1.6-W1.5-TL-1, symbol TamagotchiThing:LED_Dual_AAKK
Connections:
- net at R39.2: now also D3.3 (A2), D3.4 (A1)
- net at U5.1 (~{CHRG}): now also D3.1 (K1)
- net at U5.5 (STDBY): now also D3.2 (K2)
Changed lines of the file:
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@@
+	)
+	(symbol
+		(lib_id "TamagotchiThing:LED_Dual_AAKK")
+		(at 195.58 49.53 0)
+		(unit 1)
+		(exclude_from_sim no)
+		(in_bom yes)
+		(on_board yes)
+		(dnp no)
+		(fields_autoplaced yes)
+		(property "Reference" "D3"
+			(at 195.453 38.1 0)
+			(effects
+				(font
+					(size 1.27 1.27)
+				)
+			)
+		)
+		(property "Value" "LED_Dual_KKA"
+			(at 195.453 40.64 0)
+			(effects
+				(font
+					(size 1.27 1.27)
+				)
+			)
+		)
+		(property "Footprint" "TamagotchiThing:LED-SMD_4P-L1.6-W1.5-TL-1"
+			(at 196.342 49.53 0)
+			(effects
+				(font
+					(size 1.27 1.27)
+				)
+				(hide yes)
+			)
+		)
+		(property "Datasheet" "~"
+			(at 196.342 49.53 0)
+			(effects
+				(font
+					(size 1.27 1.27)
+				)
+				(hide yes)
+			)
+		)
+		(property "Description" "Dual LED, cathodes on pins 3 and 4"
+			(at 195.58 49.53 0)
+			(effects
+				(font
+					(size 1.27 1.27)
+				)
+				(hide yes)
+			)
+		)
+		(property "LCSC" "C965839"
+			(at 195.58 49.53 0)
+			(effects
+				(font
+					(size 1.27 1.27)
+				)
+				(hide yes)
+			)
+		)
+		(pin "3"
+		)
+		(pin "1"
+		)
+		(pin "2"
+		)
+		(pin "4"
+		)
+		(instances
+			(project ""
+				(path "/12313484-12fb-46bc-b1d8-af4ffc4cdc53/fb85a431-6246-4f25-9bf0-d572b0a7405d"
+					(reference "D3")
+					(unit 1)
+				)
+			)
+		)
 	)
 	(symbol
@@
 					(unit 1)
 				)
-			)
-		)
-	)
-	(symbol
-		(lib_id "Device:LED_Dual_AAKK")
-		(at 195.58 49.53 0)
-		(unit 1)
-		(exclude_from_sim no)
-		(in_bom yes)
-		(on_board yes)
-		(dnp no)
-		(fields_autoplaced yes)
-		(property "Reference" "D3"
-			(at 195.453 38.1 0)
-			(effects
-				(font
-					(size 1.27 1.27)
-				)
-			)
-		)
-		(property "Value" "LED_Dual_KKA"
-			(at 195.453 40.64 0)
-			(effects
-				(font
-					(size 1.27 1.27)
-				)
-			)
-		)
-		(property "Footprint" "TamagotchiThing:LED-SMD_4P-L1.6-W1.5-TL-1"
-			(at 196.342 49.53 0)
-			(effects
-				(font
-					(size 1.27 1.27)
-				)
-				(hide yes)
-			)
-		)
-		(property "Datasheet" "~"
-			(at 196.342 49.53 0)
-			(effects
-				(font
-					(size 1.27 1.27)
-				)
-				(hide yes)
-			)
-		)
-		(property "Description" "Dual LED, cathodes on pins 3 and 4"
-			(at 195.58 49.53 0)
-			(effects
-				(font
-					(size 1.27 1.27)
-				)
-				(hide yes)
-			)
-		)
-		(property "LCSC" "C965839"
-			(at 195.58 49.53 0)
-			(effects
-				(font
-					(size 1.27 1.27)
-				)
-				(hide yes)
-			)
-		)
-		(pin "2"
-		)
-		(pin "3"
-		)
-		(pin "1"
-		)
-		(pin "4"
-		)
-		(instances
-			(project ""
-				(path "/12313484-12fb-46bc-b1d8-af4ffc4cdc53/fb85a431-6246-4f25-9bf0-d572b0a7405d"
-					(reference "D3")
-					(unit 1)
-				)

Commit message: Final touches. Exported production files
Parts:
- BT1: LCSC C70377 -> (none); now left out of the parts list
- C24: LCSC (none) -> C2180552
- C25, C27: value 10u -> 10uF; Voltage (none) -> 6.3
- C26: value 22u -> 22uF; Voltage (none) -> 6.3
- Q5: LCSC (none) -> C2830320
- R33: LCSC (none) -> C60491
- R34: LCSC (none) -> C106231
- R35: LCSC (none) -> C106232
- R36: LCSC (none) -> C106235
- R39: LCSC (none) -> C60488
- R42: LCSC (none) -> C185451
- U3: LCSC (none) -> C2927799
- U5: LCSC (none) -> C725791
Changed lines of the file:
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@@
+			)
+		)
+		(property "LCSC" "C106232"
+			(at 57.15 36.83 0)
+			(effects
+				(font
+					(size 1.27 1.27)
+				)
+				(hide yes)
 			)
 		)
@@
 			)
 		)
+		(property "LCSC" "C106231"
+			(at 35.56 82.55 90)
+			(effects
+				(font
+					(size 1.27 1.27)
+				)
+				(hide yes)
+			)
+		)
 		(pin "1"
 		)
@@
 			)
 		)
-		(property "Value" "10u"
+		(property "Value" "10uF"
 			(at 62.23 144.7862 0)
 			(effects
@@
 		)
 		(property "LCSC" "C95839"
+			(at 59.69 143.51 0)
+			(effects
+				(font
+					(size 1.27 1.27)
+				)
+				(hide yes)
+			)
+		)
+		(property "Voltage" "6.3"
 			(at 59.69 143.51 0)
 			(effects
@@
 			)
 		)
+		(property "LCSC" "C60488"
+			(at 179.07 45.72 0)
+			(effects
+				(font
+					(size 1.27 1.27)
+				)
+				(hide yes)
+			)
+		)
 		(pin "1"
 		)
@@
 			)
 		)
+		(property "LCSC" "C2927799"
+			(at 78.74 44.45 0)
+			(effects
+				(font
+					(size 1.27 1.27)
+				)
+				(hide yes)
+			)
+		)
 		(pin "5"
 		)
@@
 			)
 		)
+		(property "LCSC" "C725791"
+			(at 218.44 49.53 0)
+			(effects
+				(font
+					(size 1.27 1.27)
+				)
+				(hide yes)
+			)
+		)
 		(pin "2"
 		)
@@
 			)
 		)
+		(property "LCSC" "C185451"
+			(at 238.76 55.88 0)
+			(effects
+				(font
+					(size 1.27 1.27)
+				)
+				(hide yes)
+			)
+		)
 		(pin "1"
 		)
@@
 			)
 		)
-		(property "Value" "22u"
+		(property "Value" "22uF"
 			(at 129.54 146.0563 0)
 			(effects
@@
 		)
 		(property "LCSC" "C59461"
+			(at 127 144.78 0)
+			(effects
+				(font
+					(size 1.27 1.27)
+				)
+				(hide yes)
+			)
+		)
+		(property "Voltage" "6.3"
 			(at 127 144.78 0)
 			(effects
@@
 			)
 		)
-		(property "LCSC" ""
+		(property "LCSC" "C60491"
 			(at 22.86 143.51 0)
 			(effects
@@
 		(unit 1)
 		(exclude_from_sim no)
-		(in_bom yes)
+		(in_bom no)
 		(on_board yes)
 		(dnp no)
@@
 			)
 		)
-		(property "LCSC" "C70377"
+		(property "LCSC" ""
 			(at 40.64 49.53 0)
 			(effects
@@
 			)
 		)
+		(property "LCSC" "C2180552"
+			(at 57.15 44.45 0)
+			(effects
+				(font
+					(size 1.27 1.27)
+				)
+				(hide yes)
+			)
+		)
 		(pin "1"
 		)
@@
 			)
 		)
-		(property "Value" "10u"
+		(property "Value" "10uF"
 			(at 165.1 63.5062 0)
 			(effects
@@
 		)
 		(property "LCSC" "C95839"
+			(at 162.56 62.23 0)
+			(effects
+				(font
+					(size 1.27 1.27)
+				)
+				(hide yes)
+			)
+		)
+		(property "Voltage" "6.3"
 			(at 162.56 62.23 0)
 			(effects
@@
 			)
 		)
+		(property "LCSC" "C106235"
+			(at 100.33 52.07 0)
+			(effects
+				(font
+					(size 1.27 1.27)
+				)
+				(hide yes)
+			)
+		)
 		(pin "1"
 		)
@@
 			(effects
 				(font
+					(size 1.27 1.27)
+				)
+				(hide yes)
+			)
+		)
+		(property "LCSC" "C2830320"
+			(at 78.74 63.5 90)
+			(effects
+				(font
