File: Hardware/Tamagotchi-thing/sch/OLED.kicad_sch (KiCad schematic)
At the start: 18 parts, among them J1 Conn_01x30, J5 Conn_01x14, Q2 BSS138

Commit message: schematic work
Parts:
- R8: symbol Device:R_Small -> Device:R_Small_US; LCSC C25744 -> (none)
Changed lines of the file:
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@@
 	)
 	(symbol
-		(lib_id "Device:R_Small")
+		(lib_id "Device:R_Small_US")
 		(at 74.93 68.58 0)
 		(unit 1)
@@
 			)
 		)
-		(property "Description" ""
+		(property "Description" "Resistor, small US symbol"
 			(at 74.93 68.58 0)
 			(effects
@@
 					(size 1.27 1.27)
 				)
-			)
-		)
-		(property "LCSC" "C25744"
+				(hide yes)
+			)
+		)
+		(property "LCSC" ""
 			(at 74.93 68.58 0)
 			(effects
@@
 		(at 242.57 87.63 0)
 		(unit 1)
-		(exclude_from_sim yes)
+		(exclude_from_sim no)
 		(in_bom no)
 		(on_board yes)

Commit message: Schematic work
Parts:
- added C24, C25, C26: 1uF, Capacitor_SMD:C_0402_1005Metric, symbol Device:C_Small
- added J4: Conn_01x30, TamagotchiThing:FFC-SMD_12P-P0.50_FH34SRJ-12S-0.5SH, symbol Connector_Generic_MountingPin:Conn_01x12_MountingPin
- added J7: Conn_01x14, OpenTama:LCD_14p_0.6mm, symbol Connector_Generic:Conn_01x02
- added Q6: BSS138, Package_TO_SOT_SMD:SOT-23, symbol Transistor_FET:BSS138
- added R1, R39, R40: 10k, Resistor_SMD:R_0402_1005Metric, symbol Device:R_Small_US
- added R41: 100k, Resistor_SMD:R_0402_1005Metric, symbol Device:R_Small_US
- added R7: 15, Resistor_SMD:R_0603_1608Metric, symbol Device:R_Small_US
Connections:
- net 3V3: now also J4.7 (Pin_7), R39.1, R40.1, R7.2
- net GND: now also C24.2, J4.6 (Pin_6), J4.MP (MountPin), Q6.2 (S), R1.2, R41.2
- new net: J7.1 (Pin_1), R7.1
- new net: C26.1, J4.4 (Pin_4)
- new net: C26.2, J4.5 (Pin_5)
- new net: J7.2 (Pin_2), Q6.3 (D)
- new net: C24.1, J4.1 (Pin_1)
- new net: C25.1, J4.2 (Pin_2)
- new net: C25.2, J4.3 (Pin_3)
- new net LCD2.SCL: J4.9 (Pin_9), R40.2
- new net LCD2.SDA: J4.8 (Pin_8), R39.2
- new net LCD2_A0: J4.10 (Pin_10)
- new net LCD2_BL_EN: Q6.1 (G), R1.1
- new net LCD2_CS: J4.12 (Pin_12), R41.1
- new net LCD2_RES: J4.11 (Pin_11)
Other:
- note added: "LCD2 - C18198252"

Commit message: Schematic and layout work
Parts:
- C2: renamed from C5; footprint Capacitor_SMD:C_0402_1005Metric -> Capacitor_SMD:C_0603_1608Metric
- C3: renamed from C15; footprint Capacitor_SMD:C_0402_1005Metric -> Capacitor_SMD:C_0603_1608Metric
- C4: renamed from C24; footprint Capacitor_SMD:C_0402_1005Metric -> Capacitor_SMD:C_0603_1608Metric
- C5: renamed from C25; footprint Capacitor_SMD:C_0402_1005Metric -> Capacitor_SMD:C_0603_1608Metric
- C6: renamed from C26; footprint Capacitor_SMD:C_0402_1005Metric -> Capacitor_SMD:C_0603_1608Metric
- J5: renamed from J1; footprint Bongo-Cat-Fidget-Toy:sh1106-1.3inch-oled -> TamagotchiThing:sh1106-1.3inch-oled
- R2: renamed from R1; footprint Resistor_SMD:R_0402_1005Metric -> Resistor_SMD:R_0603_1608Metric
- R3: renamed from R39; footprint Resistor_SMD:R_0402_1005Metric -> Resistor_SMD:R_0603_1608Metric
- R4: renamed from R40; footprint Resistor_SMD:R_0402_1005Metric -> Resistor_SMD:R_0603_1608Metric
- R5: renamed from R8; footprint Resistor_SMD:R_0402_1005Metric -> Resistor_SMD:R_0603_1608Metric
- R6: renamed from R41; footprint Resistor_SMD:R_0402_1005Metric -> Resistor_SMD:R_0603_1608Metric
- renumbered C4 to C1, C11 to C10, C13 to C11, C9 to C12, C10 to C7, C12 to C8, C8 to C9, J7 to J1, J5 to J2, J4 to J3, J5 to J4, Q6 to Q1, R7 to R1, R11 to R10, R101 to R7, R13 to R8, R12 to R9
Other:
- company: (none) -> Afonso Muralha
- title: (none) -> OLED

Commit message: Schematic and layout work
Parts:
- C1: footprint Capacitor_SMD:C_0603_1608Metric -> Capacitor_SMD:C_0402_1005Metric; LCSC C1615 -> (none); now not fitted; now left out of the parts list
- C10, C11, C12, C7, C8, C9: footprint Capacitor_SMD:C_0603_1608Metric -> Capacitor_SMD:C_0402_1005Metric; LCSC C23630 -> (none)
- C2, C3: footprint Capacitor_SMD:C_0603_1608Metric -> Capacitor_SMD:C_0402_1005Metric; LCSC C12530 -> (none); now not fitted; now left out of the parts list
- C4, C5, C6: footprint Capacitor_SMD:C_0603_1608Metric -> Capacitor_SMD:C_0402_1005Metric
- J2: footprint OpenTama:Hirose_FH34SRJ-14S-0.5SH_1x14-1MP_P0.50mm_Horizontal -> TamagotchiThing:Hirose_FH34SRJ-14S-0.5SH_1x14-1MP_P0.50mm_Horizontal; now not fitted; now left out of the parts list
- J4: footprint OpenTama:LCD_14p_0.6mm -> TamagotchiThing:LCD_14p_0.6mm; now not fitted; now left out of the parts list
- J5: footprint TamagotchiThing:sh1106-1.3inch-oled -> TamagotchiThing:sh1106-1.3inch-oled_1
- Q2: now not fitted; now left out of the parts list
- R1: footprint Resistor_SMD:R_0603_1608Metric -> Resistor_SMD:R_0402_1005Metric; LCSC C23150 -> (none)
- R10: footprint Resistor_SMD:R_0603_1608Metric -> Capacitor_SMD:C_0402_1005Metric; LCSC C23150 -> (none)
- R2, R3, R4, R6: footprint Resistor_SMD:R_0603_1608Metric -> Resistor_SMD:R_0402_1005Metric
- R5: footprint Resistor_SMD:R_0603_1608Metric -> Resistor_SMD:R_0402_1005Metric; now not fitted; now left out of the parts list
- R7: footprint Resistor_SMD:R_0603_1608Metric -> Resistor_SMD:R_0402_1005Metric; LCSC C25803 -> (none)
- R8, R9: footprint Resistor_SMD:R_0603_1608Metric -> Capacitor_SMD:C_0402_1005Metric; LCSC C23162 -> (none)
Changed lines of the file:
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@@
 		(unit 1)
 		(exclude_from_sim no)
-		(in_bom yes)
-		(on_board yes)
-		(dnp no)
+		(in_bom no)
+		(on_board no)
+		(dnp yes)
 		(property "Reference" "C3"
 			(at 67.1068 81.3816 0)
@@
 			)
 		)
-		(property "Footprint" "Capacitor_SMD:C_0603_1608Metric"
+		(property "Footprint" "Capacitor_SMD:C_0402_1005Metric"
 			(at 64.77 82.55 0)
 			(effects
@@
 			)
 		)
-		(property "LCSC" "C12530"
+		(property "LCSC" ""
 			(at 64.77 82.55 0)
 			(effects
@@
 		(unit 1)
 		(exclude_from_sim no)
-		(in_bom yes)
-		(on_board yes)
-		(dnp no)
+		(in_bom no)
+		(on_board no)
+		(dnp yes)
 		(property "Reference" "J4"
 			(at 127.762 90.3732 0)
@@
 			)
 		)
-		(property "Footprint" "OpenTama:LCD_14p_0.6mm"
+		(property "Footprint" "TamagotchiThing:LCD_14p_0.6mm"
 			(at 125.73 90.17 0)
 			(effects
@@
 		(unit 1)
 		(exclude_from_sim no)
-		(in_bom yes)
-		(on_board yes)
-		(dnp no)
+		(in_bom no)
+		(on_board no)
+		(dnp yes)
 		(property "Reference" "R5"
 			(at 76.4286 67.4116 0)
@@
 			)
 		)
-		(property "Footprint" "Resistor_SMD:R_0603_1608Metric"
+		(property "Footprint" "Resistor_SMD:R_0402_1005Metric"
 			(at 74.93 68.58 0)
 			(effects
@@
 			)
 		)
-		(property "Footprint" "Capacitor_SMD:C_0603_1608Metric"
+		(property "Footprint" "Capacitor_SMD:C_0402_1005Metric"
 			(at 217.17 120.65 0)
 			(effects
@@
 			)
 		)
-		(property "LCSC" "C23630"
+		(property "LCSC" ""
 			(at 217.17 120.65 0)
 			(effects
@@
 			)
 		)
-		(property "Footprint" "Resistor_SMD:R_0603_1608Metric"
+		(property "Footprint" "Resistor_SMD:R_0402_1005Metric"
 			(at 40.64 143.51 0)
 			(effects
@@
 			)
 		)
-		(property "LCSC" "C23150"
+		(property "LCSC" ""
 			(at 40.64 143.51 90)
 			(effects
@@
 			)
 		)
-		(property "Footprint" "Resistor_SMD:R_0603_1608Metric"
+		(property "Footprint" "Resistor_SMD:R_0402_1005Metric"
 			(at 63.5 175.26 0)
 			(effects
@@
 			)
 		)
-		(property "Footprint" "Resistor_SMD:R_0603_1608Metric"
+		(property "Footprint" "Capacitor_SMD:C_0402_1005Metric"
 			(at 232.41 115.57 0)
 			(effects
@@
 			)
 		)
-		(property "LCSC" "C23150"
+		(property "LCSC" ""
 			(at 232.41 115.57 90)
 			(effects
@@
 			)
 		)
-		(property "Footprint" "Capacitor_SMD:C_0603_1608Metric"
+		(property "Footprint" "Capacitor_SMD:C_0402_1005Metric"
 			(at 95.25 154.94 0)
 			(effects
@@
 		(unit 1)
 		(exclude_from_sim no)
-		(in_bom yes)
-		(on_board yes)
-		(dnp no)
+		(in_bom no)
+		(on_board no)
+		(dnp yes)
 		(property "Reference" "J2"
 			(at 102.362 90.3732 0)
@@
 			)
 		)
-		(property "Footprint" "OpenTama:Hirose_FH34SRJ-14S-0.5SH_1x14-1MP_P0.50mm_Horizontal"
+		(property "Footprint" "TamagotchiThing:Hirose_FH34SRJ-14S-0.5SH_1x14-1MP_P0.50mm_Horizontal"
 			(at 100.33 90.17 0)
 			(effects
@@
 			)
 		)
-		(property "Footprint" "Resistor_SMD:R_0603_1608Metric"
+		(property "Footprint" "Resistor_SMD:R_0402_1005Metric"
 			(at 193.04 82.55 0)
 			(effects
@@
 			)
 		)
-		(property "LCSC" "C25803"
+		(property "LCSC" ""
 			(at 193.04 82.55 0)
 			(effects
@@
 			)
 		)
-		(property "Footprint" "Capacitor_SMD:C_0603_1608Metric"
+		(property "Footprint" "Capacitor_SMD:C_0402_1005Metric"
 			(at 223.52 74.93 0)
 			(effects
@@
 			)
 		)
-		(property "LCSC" "C23630"
+		(property "LCSC" ""
 			(at 223.52 74.93 0)
 			(effects
@@
 			)
 		)
-		(property "Footprint" "Capacitor_SMD:C_0603_1608Metric"
+		(property "Footprint" "Capacitor_SMD:C_0402_1005Metric"
 			(at 226.06 123.19 0)
 			(effects
@@
 			)
 		)
-		(property "LCSC" "C23630"
+		(property "LCSC" ""
 			(at 226.06 123.19 0)
 			(effects
@@
 			)
 		)
-		(property "Footprint" "Resistor_SMD:R_0603_1608Metric"
+		(property "Footprint" "Capacitor_SMD:C_0402_1005Metric"
 			(at 201.93 113.03 0)
 			(effects
@@
 			)
 		)
-		(property "LCSC" "C23162"
+		(property "LCSC" ""
 			(at 201.93 113.03 0)
 			(effects
@@
 			)
 		)
-		(property "Footprint" "Resistor_SMD:R_0603_1608Metric"
+		(property "Footprint" "Capacitor_SMD:C_0402_1005Metric"
 			(at 194.31 113.03 0)
 			(effects
@@
 			)
 		)
-		(property "LCSC" "C23162"
+		(property "LCSC" ""
 			(at 194.31 113.03 0)
 			(effects
@@
 			)
 		)
-		(property "Footprint" "Resistor_SMD:R_0603_1608Metric"
+		(property "Footprint" "Resistor_SMD:R_0402_1005Metric"
 			(at 57.15 175.26 0)
 			(effects
@@
 			)
 		)
-		(property "Footprint" "Capacitor_SMD:C_0603_1608Metric"
+		(property "Footprint" "Capacitor_SMD:C_0402_1005Metric"
 			(at 231.14 54.61 0)
 			(effects
@@
 			)
 		)
-		(property "LCSC" "C23630"
+		(property "LCSC" ""
 			(at 231.14 54.61 90)
 			(effects
@@
 		(unit 1)
 		(exclude_from_sim no)
-		(in_bom yes)
-		(on_board yes)
-		(dnp no)
+		(in_bom no)
+		(on_board no)
+		(dnp yes)
 		(property "Reference" "Q2"
 			(at 85.1916 62.3316 0)
@@
 			)
 		)
-		(property "Footprint" "Capacitor_SMD:C_0603_1608Metric"
+		(property "Footprint" "Capacitor_SMD:C_0402_1005Metric"
 			(at 86.36 146.05 0)
 			(effects
@@
 			)
 		)
-		(property "Footprint" "TamagotchiThing:sh1106-1.3inch-oled"
+		(property "Footprint" "TamagotchiThing:sh1106-1.3inch-oled_1"
 			(at 242.57 87.63 0)
 			(effects
@@
 		(unit 1)
 		(exclude_from_sim no)
-		(in_bom yes)
-		(on_board yes)
-		(dnp no)
+		(in_bom no)
+		(on_board no)
+		(dnp yes)
 		(property "Reference" "C1"
 			(at 50.5968 80.1116 0)
@@
 			)
 		)
-		(property "Footprint" "Capacitor_SMD:C_0603_1608Metric"
+		(property "Footprint" "Capacitor_SMD:C_0402_1005Metric"
 			(at 48.26 81.28 0)
 			(effects
@@
 			)
 		)
-		(property "LCSC" "C1615"
+		(property "LCSC" ""
 			(at 48.26 81.28 0)
 			(effects
@@
 			)
 		)
-		(property "Footprint" "Capacitor_SMD:C_0603_1608Metric"
+		(property "Footprint" "Capacitor_SMD:C_0402_1005Metric"
 			(at 209.55 69.85 0)
 			(effects
@@
 			)
 		)
-		(property "LCSC" "C23630"
+		(property "LCSC" ""
 			(at 209.55 69.85 0)
 			(effects
@@
 		(unit 1)
 		(exclude_from_sim no)
-		(in_bom yes)
-		(on_board yes)
-		(dnp no)
+		(in_bom no)
+		(on_board no)
+		(dnp yes)
 		(property "Reference" "C2"
 			(at 56.9468 86.4616 0)
@@
 			)
 		)
-		(property "Footprint" "Capacitor_SMD:C_0603_1608Metric"
+		(property "Footprint" "Capacitor_SMD:C_0402_1005Metric"
 			(at 54.61 87.63 0)
 			(effects
@@
 			)
 		)
-		(property "LCSC" "C12530"
+		(property "LCSC" ""
 			(at 54.61 87.63 0)
 			(effects
@@
 			)
 		)
-		(property "Footprint" "Resistor_SMD:R_0603_1608Metric"
+		(property "Footprint" "Resistor_SMD:R_0402_1005Metric"
 			(at 46.99 156.21 0)
 			(effects
@@
 			)
 		)
-		(property "Footprint" "Resistor_SMD:R_0603_1608Metric"
+		(property "Footprint" "Resistor_SMD:R_0402_1005Metric"
 			(at 100.33 175.26 0)
 			(effects
@@
 			)
 		)
-		(property "Footprint" "Capacitor_SMD:C_0603_1608Metric"
+		(property "Footprint" "Capacitor_SMD:C_0402_1005Metric"
 			(at 95.25 148.59 0)
 			(effects
@@
 			)
 		)
-		(property "Footprint" "Capacitor_SMD:C_0603_1608Metric"
+		(property "Footprint" "Capacitor_SMD:C_0402_1005Metric"
 			(at 223.52 59.69 0)
 			(effects
@@
 			)
 		)
-		(property "LCSC" "C23630"
+		(property "LCSC" ""
 			(at 223.52 59.69 90)
 			(effects

Commit message: Schematic and Layout work
Parts:
- J1: footprint OpenTama:LCD_14p_0.6mm -> Resistor_SMD:R_1210_3225Metric; now left out of the parts list
Changed lines of the file:
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@@
 		(unit 1)
 		(exclude_from_sim no)
-		(in_bom yes)
+		(in_bom no)
 		(on_board yes)
 		(dnp no)
@@
 			)
 		)
-		(property "Footprint" "OpenTama:LCD_14p_0.6mm"
+		(property "Footprint" "Resistor_SMD:R_1210_3225Metric"
 			(at 31.75 143.51 0)
 			(effects

Commit message: Final touches. Exported production files
Parts:
- C1: value 330nF/25V -> 330nF; LCSC (none) -> C5448882; Voltage (none) -> 25
- C10, C11, C12, C7, C9: value 2.2u -> 2.2uF; LCSC (none) -> C170151; Voltage (none) -> 6.3
- C2, C3: value 2.2uF/5V -> 2.2uF; LCSC (none) -> C170151; Voltage (none) -> 6.3
- C8: value 4.7u -> 4.7uF; LCSC (none) -> C23733
- R1: LCSC (none) -> C105871
- R10: LCSC (none) -> C163467
- R2, R3, R4, R5: LCSC (none) -> C60490
- R6, R7: LCSC (none) -> C60491
- R8, R9: LCSC (none) -> C93943
Changed lines of the file:
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@@
 			)
 		)
-		(property "Value" "2.2uF/5V"
+		(property "Value" "2.2uF"
 			(at 67.1068 83.693 0)
 			(effects
@@
 			)
 		)
-		(property "LCSC" ""
+		(property "LCSC" "C170151"
 			(at 64.77 82.55 0)
 			(effects
@@
 			)
 		)
+		(property "Voltage" "6.3"
+			(at 64.77 82.55 0)
+			(effects
+				(font
+					(size 1.27 1.27)
+				)
+				(hide yes)
+			)
+		)
 		(pin "1"
 		)
@@
 			)
 		)
-		(property "LCSC" ""
+		(property "LCSC" "C60490"
 			(at 74.93 68.58 0)
 			(effects
@@
 			)
 		)
-		(property "Value" "4.7u"
+		(property "Value" "4.7uF"
 			(at 219.71 121.9135 0)
 			(effects
@@
 			)
 		)
-		(property "LCSC" ""
+		(property "LCSC" "C23733"
 			(at 217.17 120.65 0)
 			(effects
@@
 			)
 		)
-		(property "LCSC" ""
+		(property "LCSC" "C105871"
 			(at 40.64 143.51 90)
 			(effects
@@
 			)
 		)
-		(property "LCSC" ""
+		(property "LCSC" "C60490"
 			(at 63.5 175.26 0)
 			(effects
@@
 			)
 		)
-		(property "LCSC" ""
+		(property "LCSC" "C163467"
 			(at 232.41 115.57 90)
 			(effects
@@
 			)
 		)
-		(property "LCSC" ""
+		(property "LCSC" "C60491"
 			(at 193.04 82.55 0)
 			(effects
@@
 			)
 		)
-		(property "Value" "2.2u"
+		(property "Value" "2.2uF"
 			(at 226.06 76.1935 0)
 			(effects
@@
 			)
 		)
-		(property "LCSC" ""
+		(property "LCSC" "C170151"
+			(at 223.52 74.93 0)
+			(effects
+				(font
+					(size 1.27 1.27)
+				)
+				(hide yes)
+			)
+		)
+		(property "Voltage" "6.3"
 			(at 223.52 74.93 0)
 			(effects
@@
 			)
 		)
-		(property "Value" "2.2u"
+		(property "Value" "2.2uF"
 			(at 228.6 124.4535 0)
 			(effects
@@
 			)
 		)
-		(property "LCSC" ""
+		(property "LCSC" "C170151"
+			(at 226.06 123.19 0)
+			(effects
+				(font
+					(size 1.27 1.27)
+				)
+				(hide yes)
+			)
+		)
+		(property "Voltage" "6.3"
 			(at 226.06 123.19 0)
 			(effects
@@
 			)
 		)
-		(property "LCSC" ""
+		(property "LCSC" "C93943"
 			(at 201.93 113.03 0)
 			(effects
@@
 			)
 		)
-		(property "LCSC" ""
+		(property "LCSC" "C93943"
 			(at 194.31 113.03 0)
 			(effects
@@
 			)
 		)
-		(property "LCSC" ""
+		(property "LCSC" "C60490"
 			(at 57.15 175.26 0)
 			(effects
@@
 			)
 		)
-		(property "Value" "2.2u"
+		(property "Value" "2.2uF"
 			(at 231.1463 50.8 90)
 			(effects
@@
 			)
 		)
-		(property "LCSC" ""
+		(property "LCSC" "C170151"
+			(at 231.14 54.61 90)
+			(effects
+				(font
+					(size 1.27 1.27)
+				)
+				(hide yes)
+			)
+		)
+		(property "Voltage" "6.3"
 			(at 231.14 54.61 90)
 			(effects
@@
 			)
 		)
-		(property "Value" "330nF/25V"
+		(property "Value" "330nF"
 			(at 50.5968 82.423 0)
 			(effects
@@
 			)
 		)
-		(property "LCSC" ""
+		(property "LCSC" "C5448882"
 			(at 48.26 81.28 0)
 			(effects
@@
 			)
 		)
+		(property "Voltage" "25"
+			(at 48.26 81.28 0)
+			(effects
+				(font
+					(size 1.27 1.27)
+				)
+				(hide yes)
+			)
+		)
 		(pin "1"
 		)
@@
 			)
 		)
-		(property "Value" "2.2u"
+		(property "Value" "2.2uF"
 			(at 212.09 71.1135 0)
 			(effects
@@
 			)
 		)
-		(property "LCSC" ""
+		(property "LCSC" "C170151"
+			(at 209.55 69.85 0)
+			(effects
+				(font
+					(size 1.27 1.27)
+				)
+				(hide yes)
+			)
+		)
+		(property "Voltage" "6.3"
 			(at 209.55 69.85 0)
 			(effects
@@
 			)
 		)
-		(property "Value" "2.2uF/5V"
+		(property "Value" "2.2uF"
 			(at 56.9468 88.773 0)
 			(effects
@@
 			)
 		)
-		(property "LCSC" ""
+		(property "LCSC" "C170151"
 			(at 54.61 87.63 0)
 			(effects
@@
 			)
 		)
+		(property "Voltage" "6.3"
+			(at 54.61 87.63 0)
+			(effects
+				(font
+					(size 1.27 1.27)
+				)
+				(hide yes)
+			)
+		)
 		(pin "1"
 		)
@@
 			)
 		)
-		(property "LCSC" ""
+		(property "LCSC" "C60490"
 			(at 46.99 156.21 0)
 			(effects
@@
 			)
 		)
-		(property "LCSC" ""
+		(property "LCSC" "C60491"
 			(at 100.33 175.26 0)
 			(effects
@@
 			)
 		)
-		(property "Value" "2.2u"
+		(property "Value" "2.2uF"
 			(at 223.5263 55.88 90)
 			(effects
@@
 			)
 		)
-		(property "LCSC" ""
+		(property "LCSC" "C170151"
+			(at 223.52 59.69 90)
+			(effects
+				(font
+					(size 1.27 1.27)
+				)
+				(hide yes)
+			)
+		)
+		(property "Voltage" "6.3"
 			(at 223.52 59.69 90)
 			(effects

Commit message: Minor fixes. Added via stitching. BOM adjustments. Sent to production
Parts:
- C4, C5, C6: LCSC (none) -> C29266
Changed lines of the file:
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@@
 			)
 		)
-		(property "LCSC" ""
+		(property "LCSC" "C29266"
 			(at 95.25 154.94 0)
 			(effects
@@
 			)
 		)
-		(property "LCSC" ""
+		(property "LCSC" "C29266"
 			(at 86.36 146.05 0)
 			(effects
@@
 			)
 		)
-		(property "LCSC" ""
+		(property "LCSC" "C29266"
 			(at 95.25 148.59 0)
 			(effects
